File: geiger_clock/geiger_module.sch (EAGLE design)
At the start: 39 parts, among them IC2 7805TV, IC3 74125N, Q1 FJN3303F, Q2 2N3904, Q3 2N3904, U1 TLC555CP, U2 ATTINY2313, X1 8MHz

Commit message: updated the geiger module
Parts:
- removed C5: 10uF, capacitor-wima:C2.5/2
- removed IC1: (no value), v-reg-3:LM1117V
- added H1: MOUNT-HOLE3.2, holes:MOUNT-HOLE3.2
- added JP1: (no value), arduino_jw:ARDUINO_CONN-ICSP
- added JP2: (no value), pinhead:PINHD-1X6
- added Q4: BSS138, bss138_10:BSS138
- added R12, R13: 10k, resistor:R-US_0207/10
- C4: device capacitor-wima:C2.5/2 -> SparkFun-Capacitors:10UF-POLAR-RADIAL-2.5MM-25V-20%
- IC3: value 74125N -> LM1117T(V)-3.3; device 74xx-us:74125N -> lm1117_10:LM1117T(V)-3.3
Connections:
- new net N$13: JP1.1, U2.(MISO)PB6
- new net N$16: JP1.4, U2.(MOSI)PB5
- new net N$5: JP1.3, U2.(UCSK)PB7
- new net N$6: JP2.2, U2.(TXD)PD1
- new net N$7: JP2.3, U2.(RXD)PD0
- net 5V: now also IC3.IN, R13.2; no longer C4.1, IC1.IN, IC3P.VCC
- net GND: now also C4.-, IC3.GND, JP1.6, JP2.5, JP2.6; no longer C4.2, C5.2, IC1.GND, IC3A.OE, IC3P.GND
- net N$2: now also JP1.5
- net PIN16: now also Q4.S, R12.1; no longer IC3A.I
- net PIN165V: now also Q4.D, R13.1; no longer IC3A.O
- net VCC: now also C4.+, IC3.OUT, JP1.2, Q4.G, R12.2; no longer C5.1, IC1.OUT
