File: milkdrop/projectm_eurorack/projectm_eurorack.kicad_pcb (KiCad board)
At the start: 2 copper layers, 75 x 100 mm, 59 parts, among them J1 Micro_SD_Card, J2 Conn_02x05_Odd_Even, J3 AudioJack3_SwitchT, J4 USB_A, J5 AudioJack3_SwitchT, J6 690-019-298-412, J7 Barrel_Jack_Switch, Q1 MMBT3904, SW1 SW_Push, U1 RT9742SNGV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

Commit message: Added missing base resistor
Parts:
- added R12: 2.2k, Resistor_SMD:R_0603_1608Metric, F.Cu at (10.2, 94.2)
Connections:
- SW1 pad 2: Net-(Q1-B) -> Net-(R12-Pad2)
Routing:
- net GND: track 232.2 -> 211.7 mm
- net Net-(R12-Pad2): track 0.00 -> 8.19 mm
- net Net-(Q1-B): track 13.3 -> 5.83 mm
