File: noise_toaster/pcb/noise_toaster.kicad_sch (KiCad schematic)
At the start: 133 parts, among them J1 Thonk, J2 Conn_01x02, J3 Thonk, J4 Thonk, Q1 MMBT3904, Q10 MMBT5457, Q2 MMBT3904, Q3 MMBT5457, Q4 MMBT3904, Q5 MMBT3904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

Commit message: Fixed potentiometer polarities
Connections:
- net BN: now also RV1.1, RV2.1; no longer RV1.3, RV2.3
- net BP: now also RV1.3; no longer RV1.1
- net GND: now also RV3.1; no longer RV3.3
- net LFO: now also RV2.3; no longer RV2.1
- net at R32.2: now also RV6.1; no longer RV6.3
- net at SW4.2 (B): now also RV6.3; no longer RV6.1
- net at SW1.1 (A): now also RV3.3; no longer RV3.1
Changed lines of the file:
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@@
     (stroke (width 0) (type default))
   )
+  (wire (pts (xy 36.83 144.78) (xy 36.83 151.13))
+    (stroke (width 0) (type default))
+  )
   (wire (pts (xy 228.6 77.47) (xy 231.14 77.47))
     (stroke (width 0) (type default))
@@
     (stroke (width 0) (type default))
   )
-  (wire (pts (xy 36.83 151.13) (xy 36.83 144.78))
-    (stroke (width 0) (type default))
-  )
   (wire (pts (xy 120.65 24.13) (xy 120.65 25.4))
     (stroke (width 0) (type default))
@@
     )
   )
-  (symbol (lib_id "Device:R_Potentiometer_US") (at 25.4 45.72 0) (unit 1)
-    (in_bom yes) (on_board yes) (dnp no) (fields_autoplaced)
-    (property "Reference" "RV2" (at 22.86 44.45 0)
+  (symbol (lib_id "Device:R_Potentiometer_US") (at 25.4 45.72 0) (mirror x) (unit 1)
+    (in_bom yes) (on_board yes) (dnp no)
+    (property "Reference" "RV2" (at 22.86 46.99 0)
       (effects (font (size 1.27 1.27)) (justify right))
     )
-    (property "Value" "100k" (at 22.86 46.99 0)
+    (property "Value" "100k" (at 22.86 44.45 0)
       (effects (font (size 1.27 1.27)) (justify right))
     )
@@
     )
   )
-  (symbol (lib_id "Device:R_Potentiometer_US") (at 36.83 140.97 0) (unit 1)
-    (in_bom yes) (on_board yes) (dnp no) (fields_autoplaced)
-    (property "Reference" "RV6" (at 34.29 139.7 0)
+  (symbol (lib_id "Device:R_Potentiometer_US") (at 36.83 140.97 0) (mirror x) (unit 1)
+    (in_bom yes) (on_board yes) (dnp no)
+    (property "Reference" "RV6" (at 34.29 142.24 0)
       (effects (font (size 1.27 1.27)) (justify right))
     )
-    (property "Value" "100k" (at 34.29 142.24 0)
+    (property "Value" "100k" (at 34.29 139.7 0)
       (effects (font (size 1.27 1.27)) (justify right))
     )
@@
     )
   )
-  (symbol (lib_id "Device:R_Potentiometer_US") (at 25.4 66.04 0) (unit 1)
-    (in_bom yes) (on_board yes) (dnp no) (fields_autoplaced)
-    (property "Reference" "RV3" (at 22.86 64.77 0)
+  (symbol (lib_id "Device:R_Potentiometer_US") (at 25.4 66.04 0) (mirror x) (unit 1)
+    (in_bom yes) (on_board yes) (dnp no)
+    (property "Reference" "RV3" (at 22.86 67.31 0)
       (effects (font (size 1.27 1.27)) (justify right))
     )
-    (property "Value" "100k" (at 22.86 67.31 0)
+    (property "Value" "100k" (at 22.86 64.77 0)
       (effects (font (size 1.27 1.27)) (justify right))
     )
@@
     )
   )
-  (symbol (lib_id "Device:R_Potentiometer_US") (at 25.4 24.13 0) (unit 1)
-    (in_bom yes) (on_board yes) (dnp no) (fields_autoplaced)
-    (property "Reference" "RV1" (at 22.86 22.86 0)
+  (symbol (lib_id "Device:R_Potentiometer_US") (at 25.4 24.13 0) (mirror x) (unit 1)
+    (in_bom yes) (on_board yes) (dnp no)
+    (property "Reference" "RV1" (at 22.86 25.4 0)
       (effects (font (size 1.27 1.27)) (justify right))
     )
-    (property "Value" "100k" (at 22.86 25.4 0)
+    (property "Value" "100k" (at 22.86 22.86 0)
       (effects (font (size 1.27 1.27)) (justify right))
     )
