File: power_bus/power_bus.kicad_pcb (KiCad board)
At the start: 2 copper layers, 450 x 40 mm, 28 parts, among them J1 Conn_02x08_Odd_Even, J10 Conn_02x08_Odd_Even, J11 Conn_02x08_Odd_Even, J12 Conn_02x08_Odd_Even, J13 Conn_02x08_Odd_Even, J14 Conn_02x08_Odd_Even, J15 Conn_02x08_Odd_Even, J16 Conn_02x08_Odd_Even, J17 Conn_02x08_Odd_Even, J18 Conn_02x08_Odd_Even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

Commit message: Added mega_12v_pwr
Parts:
- added J23: Conn_01x01, AlexCustom:SPADE, F.Cu at (521.2, 187.9)
- added J24: Conn_01x01, AlexCustom:SPADE, F.Cu at (521.2, 202.9)
- added J25: Conn_01x01, AlexCustom:SPADE, F.Cu at (521.2, 207.9)
- added J26: Conn_01x01, AlexCustom:SPADE, F.Cu at (521.2, 212.9)
- added J27: Conn_01x01, AlexCustom:SPADE, F.Cu at (109.2, 212.9)
- added J28: Conn_01x01, AlexCustom:SPADE, F.Cu at (109.2, 207.9)
- added J29: Conn_01x01, AlexCustom:SPADE, F.Cu at (109.2, 202.9)
- added J30: Conn_01x01, AlexCustom:SPADE, F.Cu at (109.2, 197.9)
- added J31: Conn_01x01, AlexCustom:SPADE, F.Cu at (109.2, 192.9)
- added J32: Conn_01x01, AlexCustom:SPADE, F.Cu at (109.2, 187.9)
- J21, J22: value Screw_Terminal_01x06 -> Conn_01x01; footprint TerminalBlock_Phoenix:TerminalBlock_Phoenix_MKDS-1,5-6-5.08_1x06_P5.08mm_Horizontal -> AlexCustom:SPADE
- R1, R2, R3: footprint PCM_4ms_Resistor:R_Axial_DIN0207_L6.3mm_D2.5mm_P7.62mm_Horizontal -> Resistor_THT:R_Axial_DIN0207_L6.3mm_D2.5mm_P7.62mm_Horizontal
- moved J22 414.9 mm to (521.2, 197.9), turned to 90 degrees
- moved J21 20.9 mm to (521.2, 192.9)
- moved R1 3.81 mm to (481.2, 218.2)
- moved R3 3.80 mm to (502.9, 218.2)
- moved R2 3.70 mm to (461.0, 218.3)
Connections:
- J21 pad 1: -12V -> +12V
- J22 pad 1: +5V -> GND
Routing:
- net +5V: track 949.8 -> 948.6 mm
- net +12V: track 919.0 -> 918.2 mm
- net -12V: track 850.9 -> 850.3 mm

Commit message: Updated gerbers
Parts:
- moved D1 6.31 mm to (487.5, 218.0)
- moved D2 6.31 mm to (467.3, 218.1)
- moved D3 6.31 mm to (509.2, 218.0)
- moved R1 6.31 mm to (474.9, 218.0)
- moved R2 6.31 mm to (454.7, 218.1)
- moved R3 6.31 mm to (496.6, 218.0)
Routing:
- net +5V: track 948.6 -> 955.2 mm
- net +12V: track 918.2 -> 924.5 mm
- net -12V: track 850.3 -> 856.6 mm
Changed lines of the file:
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@@
   )
   (footprint "LED_THT:LED_D3.0mm" (layer "F.Cu")
-    (at 515.495 218.24 180)
+    (at 509.185 218.04 180)
     (descr "LED, diameter 3.0mm, 2 pins")
     (tags "LED diameter 3.0mm 2 pins")
@@
   )
   (footprint "LED_THT:LED_D3.0mm" (layer "F.Cu")
-    (at 473.595 218.34 180)
+    (at 467.285 218.14 180)
     (descr "LED, diameter 3.0mm, 2 pins")
     (tags "LED diameter 3.0mm 2 pins")
@@
   )
   (footprint "LED_THT:LED_D3.0mm" (layer "F.Cu")
-    (at 493.795 218.24 180)
+    (at 487.485 218.04 180)
     (descr "LED, diameter 3.0mm, 2 pins")
     (tags "LED diameter 3.0mm 2 pins")
@@
   )
   (footprint "Resistor_THT:R_Axial_DIN0207_L6.3mm_D2.5mm_P7.62mm_Horizontal" (layer "F.Cu")
-    (at 461.01 218.34)
+    (at 454.7 218.14)
     (descr "Resistor, Axial_DIN0207 series, Axial, Horizontal, pin pitch=7.62mm, 0.25W = 1/4W, length*diameter=6.3*2.5mm^2, http://cdn-reichelt.de/documents/datenblatt/B400/1_4W%23YAG.pdf")
     (tags "Resistor Axial_DIN0207 series Axial Horizontal pin pitch 7.62mm 0.25W = 1/4W length 6.3mm diameter 2.5mm")
@@
   )
   (footprint "Resistor_THT:R_Axial_DIN0207_L6.3mm_D2.5mm_P7.62mm_Horizontal" (layer "F.Cu")
-    (at 502.92 218.24)
+    (at 496.61 218.04)
     (descr "Resistor, Axial_DIN0207 series, Axial, Horizontal, pin pitch=7.62mm, 0.25W = 1/4W, length*diameter=6.3*2.5mm^2, http://cdn-reichelt.de/documents/datenblatt/B400/1_4W%23YAG.pdf")
     (tags "Resistor Axial_DIN0207 series Axial Horizontal pin pitch 7.62mm 0.25W = 1/4W length 6.3mm diameter 2.5mm")
@@
   )
   (footprint "Resistor_THT:R_Axial_DIN0207_L6.3mm_D2.5mm_P7.62mm_Horizontal" (layer "F.Cu")
-    (at 481.21 218.24)
+    (at 474.9 218.04)
     (descr "Resistor, Axial_DIN0207 series, Axial, Horizontal, pin pitch=7.62mm, 0.25W = 1/4W, length*diameter=6.3*2.5mm^2, http://cdn-reichelt.de/documents/datenblatt/B400/1_4W%23YAG.pdf")
     (tags "Resistor Axial_DIN0207 series Axial Horizontal pin pitch 7.62mm 0.25W = 1/4W length 6.3mm diameter 2.5mm")
@@
     (effects (font (size 1 1) (thickness 0.15)) (justify bottom))
   )
-  (gr_text "+12V" (at 497.32 218.84) (layer "F.SilkS")
+  (gr_text "+12V" (at 491.01 218.64) (layer "F.SilkS")
     (effects (font (size 1 1) (thickness 0.15)) (justify bottom))
   )
@@
     (effects (font (size 1 1) (thickness 0.15)) (justify bottom))
   )
-  (gr_text "-12V" (at 518.92 218.84) (layer "F.SilkS")
+  (gr_text "-12V" (at 512.62 218.74) (layer "F.SilkS")
     (effects (font (size 1 1) (thickness 0.15)) (justify bottom))
   )
@@
     (effects (font (size 1 1) (thickness 0.15)) (justify bottom))
   )
-  (gr_text "+5V" (at 476.42 218.84) (layer "F.SilkS")
+  (gr_text "+5V" (at 470.11 218.64) (layer "F.SilkS")
     (effects (font (size 1 1) (thickness 0.15)) (justify bottom))
   )
@@
     (effects (font (size 1 1) (thickness 0.15)) (justify bottom))
   )
-  (segment (start 488.83 218.24) (end 491.255 218.24) (width 0.25) (layer "F.Cu") (net 2))
-  (segment (start 471.055 218.34) (end 468.52 218.34) (width 0.25) (layer "F.Cu") (net 3))
+  (segment (start 482.52 218.04) (end 484.945 218.04) (width 0.25) (layer "F.Cu") (net 2))
+  (segment (start 464.745 218.14) (end 462.21 218.14) (width 0.25) (layer "F.Cu") (net 3))
   (segment (start 123.38 209.93) (end 114.77 209.93) (width 1) (layer "F.Cu") (net 4))
   (segment (start 523.76 212.94) (end 523.81 212.99) (width 0.25) (layer "F.Cu") (net 4))
@@
   (segment (start 515.67 209.93) (end 518.68 212.94) (width 1) (layer "F.Cu") (net 4))
   (segment (start 123.38 209.93) (end 505.92 209.93) (width 1) (layer "F.Cu") (net 4))
-  (segment (start 515.495 218.24) (end 518.46 218.24) (width 0.25) (layer "F.Cu") (net 4))
+  (segment (start 518.66 218.04) (end 523.76 212.94) (width 0.25) (layer "F.Cu") (net 4))
   (segment (start 523.81 212.99) (end 523.81 213.64) (width 0.25) (layer "F.Cu") (net 4))
   (segment (start 505.92 209.93) (end 515.67 209.93) (width 1) (layer "F.Cu") (net 4))
   (segment (start 114.77 209.93) (end 111.76 212.94) (width 1) (layer "F.Cu") (net 4))
-  (segment (start 518.46 218.24) (end 523.76 212.94) (width 0.25) (layer "F.Cu") (net 4))
   (segment (start 111.76 212.94) (end 106.68 212.94) (width 1) (layer "F.Cu") (net 4))
+  (segment (start 509.185 218.04) (end 518.66 218.04) (width 0.25) (layer "F.Cu") (net 4))
   (segment (start 114.77 209.93) (end 111.76 212.94) (width 1) (layer "B.Cu") (net 4))
   (segment (start 111.76 212.94) (end 106.68 212.94) (width 1) (layer "B.Cu") (net 4))
@@
   (segment (start 123.38 209.93) (end 114.77 209.93) (width 1) (layer "B.Cu") (net 4))
   (segment (start 515.67 209.93) (end 518.68 212.94) (width 1) (layer "B.Cu") (net 4))
-  (segment (start 512.955 218.24) (end 510.53 218.24) (width 0.25) (layer "F.Cu") (net 5))
-  (segment (start 524.595 219.865) (end 526.22 218.24) (width 0.25) (layer "F.Cu") (net 6))
+  (segment (start 506.645 218.04) (end 504.22 218.04) (width 0.25) (layer "F.Cu") (net 5))
   (segment (start 118.59 199.77) (end 111.76 192.94) (width 1) (layer "F.Cu") (net 6))
+  (segment (start 476.525 219.665) (end 476.725 219.865) (width 0.25) (layer "F.Cu") (net 6))
+  (segment (start 524.595 219.865) (end 526.22 218.24) (width 0.25) (layer "F.Cu") (net 6))
   (segment (start 511.85 199.77) (end 518.68 192.94) (width 1) (layer "F.Cu") (net 6))
   (segment (start 505.92 199.77) (end 123.38 199.77) (width 1) (layer "F.Cu") (net 6))
-  (segment (start 481.21 218.24) (end 482.835 219.865) (width 0.25) (layer "F.Cu") (net 6))
-  (segment (start 518.68 192.94) (end 523.76 192.94) (width 1) (layer "F.Cu") (net 6))
-  (segment (start 482.835 219.865) (end 524.595 219.865) (width 0.25) (layer "F.Cu") (net 6))
+  (segment (start 474.9 218.04) (end 476.525 219.665) (width 0.25) (layer "F.Cu") (net 6))
   (segment (start 526.22 195.4) (end 523.76 192.94) (width 0.25) (layer "F.Cu") (net 6))
+  (segment (start 518.68 192.94) (end 523.76 192.94) (width 1) (layer "F.Cu") (net 6))
+  (segment (start 526.22 218.24) (end 526.22 195.4) (width 0.25) (layer "F.Cu") (net 6))
   (segment (start 111.76 192.94) (end 106.68 192.94) (width 1) (layer "F.Cu") (net 6))
+  (segment (start 476.725 219.865) (end 524.595 219.865) (width 0.25) (layer "F.Cu") (net 6))
   (segment (start 505.92 199.77) (end 511.85 199.77) (width 1) (layer "F.Cu") (net 6))
   (segment (start 123.38 199.77) (end 118.59 199.77) (width 1) (layer "F.Cu") (net 6))
-  (segment (start 526.22 218.24) (end 526.22 195.4) (width 0.25) (layer "F.Cu") (net 6))
   (segment (start 505.92 199.77) (end 511.85 199.77) (width 1) (layer "B.Cu") (net 6))
   (segment (start 118.59 199.77) (end 111.76 192.94) (width 1) (layer "B.Cu") (net 6))
@@
   (segment (start 505.92 197.23) (end 509.39 197.23) (width 1) (layer "F.Cu") (net 7))
   (segment (start 123.38 197.23) (end 505.92 197.23) (width 1) (layer "F.Cu") (net 7))
-  (segment (start 460.9 218.34) (end 462.875 220.315) (width 0.25) (layer "F.Cu") (net 7))
-  (segment (start 526.67 190.85) (end 523.76 187.94) (width 0.25) (layer "F.Cu") (net 7))
   (segment (start 524.781396 220.315) (end 526.67 218.426396) (width 0.25) (layer "F.Cu") (net 7))
-  (segment (start 462.875 220.315) (end 524.781396 220.315) (width 0.25) (layer "F.Cu") (net 7))
+  (segment (start 454.59 218.14) (end 456.565 220.115) (width 0.25) (layer "F.Cu") (net 7))
   (segment (start 526.67 218.426396) (end 526.67 190.85) (width 0.25) (layer "F.Cu") (net 7))
+  (segment (start 526.67 190.85) (end 523.76 187.94) (width 0.25) (layer "F.Cu") (net 7))
   (segment (start 111.76 187.94) (end 106.68 187.94) (width 1) (layer "F.Cu") (net 7))
   (segment (start 121.05 197.23) (end 111.76 187.94) (width 1) (layer "F.Cu") (net 7))
+  (segment (start 456.455 220.005) (end 456.765 220.315) (width 0.25) (layer "F.Cu") (net 7))
+  (segment (start 456.765 220.315) (end 524.781396 220.315) (width 0.25) (layer "F.Cu") (net 7))
   (segment (start 518.68 187.94) (end 523.76 187.94) (width 1) (layer "F.Cu") (net 7))
   (segment (start 123.38 197.23) (end 121.01 197.23) (width 1) (layer "B.Cu") (net 7))

Commit message: Updated resistor values
Parts:
- R1, R3: value 2.2k -> 4.7k
- R2: value 1k -> 2.2k
Changed lines of the file:
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@@
         (effects (font (size 1 1) (thickness 0.15)))
     )
-    (fp_text value "1k" (at 3.81 2.37) (layer "F.Fab")
+    (fp_text value "2.2k" (at 3.81 2.37) (layer "F.Fab")
         (effects (font (size 1 1) (thickness 0.15)))
     )
@@
         (effects (font (size 1 1) (thickness 0.15)))
     )
-    (fp_text value "2.2k" (at 3.81 2.37) (layer "F.Fab")
+    (fp_text value "4.7k" (at 3.81 2.37) (layer "F.Fab")
         (effects (font (size 1 1) (thickness 0.15)))
     )
@@
         (effects (font (size 1 1) (thickness 0.15)))
     )
-    (fp_text value "2.2k" (at 3.81 2.37) (layer "F.Fab")
-        (effects (font (size 1 1) (thickness 0.15)))
-    )
+    (fp_text value "4.7k" (at 3.81 2.37) (layer "F.Fab")
+        (effects (font (size 1 1) (thickness 0.15)))
+    )

Commit message: Moved spade connectors
Parts:
- removed J24, J25, J29, J30: Conn_01x01, AlexCustom:SPADE
- moved J22 216.1 mm to (305.2, 204.4)
- moved J21 216.0 mm to (305.2, 196.9)
- moved J23 216.0 mm to (305.2, 189.4)
- moved J26 216.0 mm to (305.2, 211.9)
- moved J31 186.0 mm to (295.2, 196.9)
- moved J28 186.0 mm to (295.2, 204.4)
- moved J32 186.0 mm to (295.2, 189.4)
- moved J27 186.0 mm to (295.2, 211.9)
- moved D3 62.9 mm to (446.3, 217.7)
- moved R3 62.9 mm to (433.8, 217.7)
- moved R2 21.0 mm to (475.7, 217.6)
- moved D2 21.0 mm to (488.2, 217.6)
- moved D1 21.0 mm to (466.5, 217.6)
- moved R1 21.0 mm to (453.9, 217.6)
- moved J14 20.2 mm to (245.7, 209.4)
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Routing:
- net +5V: track 955.2 -> 851.2 mm
- net +12V: track 924.5 -> 852.5 mm
- net -12V: track 856.6 -> 799.5 mm
- net CV: track 765.1 -> 767.8 mm
- net GATE: track 765.1 -> 762.7 mm
Other:
- board size 450 x 40 mm -> 420 x 40 mm
