File: wand_receiver/hardware/wand_receiver/wand_receiver.kicad_pcb (KiCad board)
At the start: 2 copper layers, 20 x 100 mm, 53 parts, among them J1 AudioJack2_SwitchT, J2 Conn_02x05_Odd_Even, J3 AudioJack2_SwitchT, J4 AudioJack2_SwitchT, J5 USB_C_Receptacle_USB2.0, Q2 MUN5214DW1T1G, U1 R-783.3-1.0, U2 MCP4922-ESL, U3 MCP4922-ESL, U4 LM324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

Commit message: Added electrolytic caps
Parts:
- removed C6: 10u, Capacitor_SMD:C_0603_1608Metric
- C5: value 10u -> 100u; footprint Capacitor_SMD:C_0603_1608Metric -> Capacitor_SMD:CP_Elec_6.3x5.4
- moved C9 24.1 mm to (168.7, 72.1)
- moved C7 11.4 mm to (166.2, 73.8)
- moved C8 11.4 mm to (166.2, 75.4)
- moved D2 11.4 mm to (165.4, 71.8)
- moved C16 6.54 mm to (178.1, 72.0)
- moved U1 6.44 mm to (174.7, 62.5)
- moved C5 4.61 mm to (177.2, 55.2), turned to 180 degrees
Routing:
- net +3V3: track 159.2 -> 151.6 mm
- net +12V: track 52.9 -> 57.5 mm, vias 1 -> 0
- net Net-(D2-K): track 7.99 -> 10.5 mm
- net -12V: track 28.9 -> 30.1 mm
